File: CNC-FPGA Driver PCB/CNC-FPGA Driver PCB.kicad_sch (KiCad schematic)
At the start: 6 parts, among them J1 12V_Screw_Terminal

Commit message: updated pcb traces
Parts:
- A1: value A4988 Stepper Driver -> A4988 N Axis Driver
- C1: value C_Polarized -> 100[µF]
Connections:
- net +3.3V: now also A1.10 (VDD); no longer A1.2 (VDD)
- net DIR: now also A1.8 (DIR), JA1.12 (Pin_1); no longer A1.16 (DIR), JA1.1 (Pin_1)
- net EN: now also A1.1 (~{ENABLE}); no longer A1.9 (~{ENABLE})
- net GND: now also A1.15 (GND), A1.9 (GND), J1.1 (Pin_2); no longer A1.1 (GND), A1.7 (GND), J1.2 (Pin_2)
- net LS+: now also JA1.10 (Pin_6), LimitSwitchX1.1 (C); no longer JA1.6 (Pin_6), LimitSwitchX1.3 (A)
- net LS-: now also JA1.8 (Pin_5), LimitSwitchX1.3 (A); no longer JA1.5 (Pin_5), LimitSwitchX1.1 (C)
- net LSS: now also JA1.9 (Pin_4); no longer JA1.4 (Pin_4)
- net MS1: now also A1.2 (MS1); no longer A1.10 (MS1)
- net MS1 : now also JA1.1 (Pin_8); no longer JA1.8 (Pin_8)
- net MS2: now also A1.3 (MS2), JA1.2 (Pin_9); no longer A1.11 (MS2), JA1.9 (Pin_9)
- net MS3: now also A1.4 (MS3), JA1.3 (Pin_10); no longer A1.12 (MS3), JA1.10 (Pin_10)
- net RST: now also A1.5 (~{RESET}), JA1.4 (Pin_3); no longer A1.13 (~{RESET}), JA1.3 (Pin_3)
- net SLP: now also A1.6 (~{SLEEP}), JA1.5 (Pin_12); no longer A1.14 (~{SLEEP}), JA1.12 (Pin_12)
- net STEP: now also A1.7 (STEP), JA1.6 (Pin_2); no longer A1.15 (STEP), JA1.2 (Pin_2)
- net at StepperX1.1 (Pin_1): now also A1.11 (1B); no longer A1.3 (1B)
- net at StepperX1.2 (Pin_2): now also A1.12 (1A); no longer A1.4 (1A)
- net at StepperX1.3 (Pin_3): now also A1.13 (2A); no longer A1.5 (2A)
- net at StepperX1.4 (Pin_4): now also A1.14 (2B); no longer A1.6 (2B)
- new net: A1.16 (VMOT), C1.1, J1.2 (Pin_1)
Other:
- company: (none) -> Amir Zuabi & Alex Vassiliev
- title: (none) -> CNC-FPGA Driver Board
Changed lines of the file:
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@@
 	(generator_version "9.0")
 	(paper "A4")
+	(title_block
+		(title "CNC-FPGA Driver Board")
+		(date "2025-06-24")
+		(rev "1.0")
+		(company "Amir Zuabi & Alex Vassiliev")
+	)
 	(junction
 		(at 232.41 110.49)
@@
 		)
 	)
-	(label "LS+"
+	(label "LS-"
 		(at 254 148.59 0)
 		(effects
@@
 		)
 	)
-	(label "LS-"
+	(label "LS+"
 		(at 254 153.67 0)
 		(effects
@@
 		(on_board yes)
 		(dnp no)
-		(fields_autoplaced yes)
 		(property "Reference" "JA1"
-			(at 194.31 115.57 0)
+			(at 194.31 118.618 0)
 			(effects
 				(font
@@
 					(size 1.27 1.27)
 				)
+				(hide yes)
 			)
 		)
@@
 		(pin "12"
 		)
+		(pin "9"
+		)
+		(pin "2"
+		)
+		(pin "7"
+		)
+		(pin "8"
+		)
 		(pin "5"
-		)
-		(pin "2"
-		)
-		(pin "7"
-		)
-		(pin "8"
-		)
-		(pin "9"
 		)
 		(pin "10"
@@
 			)
 		)
-		(property "Value" "A4988 Stepper Driver"
+		(property "Value" "A4988 N Axis Driver"
 			(at 238.76 117.856 0)
 			(effects
@@
 			)
 		)
+		(pin "7"
+		)
+		(pin "3"
+		)
+		(pin "1"
+		)
+		(pin "13"
+		)
+		(pin "11"
+		)
+		(pin "4"
+		)
+		(pin "15"
+		)
+		(pin "10"
+		)
+		(pin "8"
+		)
+		(pin "2"
+		)
+		(pin "14"
+		)
+		(pin "12"
+		)
+		(pin "16"
+		)
 		(pin "9"
-		)
-		(pin "3"
-		)
-		(pin "1"
-		)
-		(pin "13"
-		)
-		(pin "11"
-		)
-		(pin "4"
-		)
-		(pin "15"
-		)
-		(pin "10"
-		)
-		(pin "8"
-		)
-		(pin "2"
-		)
-		(pin "14"
-		)
-		(pin "12"
-		)
-		(pin "16"
-		)
-		(pin "7"
 		)
 		(pin "5"
@@
 			)
 		)
-		(property "Value" "C_Polarized"
+		(property "Value" "100[µF]"
 			(at 235.966 105.156 0)
 			(effects
@@
 		(on_board yes)
 		(dnp no)
-		(fields_autoplaced yes)
 		(property "Reference" "StepperX1"
-			(at 247.65 132.0799 0)
+			(at 247.65 137.414 90)
 			(effects
 				(font
@@
 				)
 				(justify left)
+				(hide yes)
 			)
 		)
@@
 				)
 				(justify left)
+				(hide yes)
 			)
 		)
@@
 		(dnp no)
 		(property "Reference" "LimitSwitchX1"
-			(at 248.92 142.24 0)
+			(at 248.92 145.288 0)
 			(effects
 				(font
@@
 					(size 1.27 1.27)
 				)
-			)
-		)
+				(hide yes)
+			)
+		)
